File: KiCAD/CoolBoard/test.kicad_sch (KiCad schematic)
At the start: 10 parts, among them J1 Screw_Terminal_01x02, J2 Screw_Terminal_01x02, J3 Screw_Terminal_01x02, J4 Conn_01x06_Pin, Q1 Q_NMOS_GDS

Commit message: updates to BOM and updates to othere boards (context of kicad pcbs)
Parts:
- A1: now left out of the parts list
Changed lines of the file:
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@@
+	)
+	(junction
+		(at 88.9 49.53)
+		(diameter 0)
+		(color 0 0 0 0)
 	)
 	(junction
@@
 	)
 	(junction
-		(at 92.71 49.53)
-		(diameter 0)
-		(color 0 0 0 0)
-	)
-	(junction
 		(at 158.75 113.03)
 		(diameter 0)
@@
 	(wire
 		(pts
-			(xy 92.71 115.57) (xy 92.71 49.53)
-		)
-		(stroke
-			(width 0)
-			(type default)
-		)
-	)
-	(wire
-		(pts
 			(xy 86.36 80.01) (xy 86.36 74.93)
 		)
@@
 	(wire
 		(pts
+			(xy 88.9 49.53) (xy 88.9 90.17)
+		)
+		(stroke
+			(width 0)
+			(type default)
+		)
+	)
+	(wire
+		(pts
 			(xy 168.91 81.28) (xy 161.29 81.28)
 		)
@@
 	(wire
 		(pts
+			(xy 90.17 119.38) (xy 154.94 119.38)
+		)
+		(stroke
+			(width 0)
+			(type default)
+		)
+	)
+	(wire
+		(pts
 			(xy 158.75 115.57) (xy 168.91 115.57)
 		)
@@
 	(wire
 		(pts
-			(xy 140.97 115.57) (xy 92.71 115.57)
-		)
-		(stroke
-			(width 0)
-			(type default)
-		)
-	)
-	(wire
-		(pts
 			(xy 168.91 76.2) (xy 168.91 67.31)
 		)
@@
 	(wire
 		(pts
+			(xy 154.94 110.49) (xy 154.94 119.38)
+		)
+		(stroke
+			(width 0)
+			(type default)
+		)
+	)
+	(wire
+		(pts
+			(xy 90.17 90.17) (xy 90.17 119.38)
+		)
+		(stroke
+			(width 0)
+			(type default)
+		)
+	)
+	(wire
+		(pts
 			(xy 78.74 78.74) (xy 85.09 78.74)
 		)
@@
 	(wire
 		(pts
+			(xy 88.9 90.17) (xy 90.17 90.17)
+		)
+		(stroke
+			(width 0)
+			(type default)
+		)
+	)
+	(wire
+		(pts
 			(xy 91.44 52.07) (xy 91.44 118.11)
 		)
@@
 	(wire
 		(pts
-			(xy 81.28 49.53) (xy 92.71 49.53)
+			(xy 81.28 49.53) (xy 88.9 49.53)
 		)
 		(stroke
@@
 	(wire
 		(pts
-			(xy 92.71 49.53) (xy 100.33 49.53)
+			(xy 88.9 49.53) (xy 100.33 49.53)
 		)
 		(stroke
@@
 	(wire
 		(pts
-			(xy 140.97 110.49) (xy 140.97 115.57)
-		)
-		(stroke
-			(width 0)
-			(type default)
-		)
-	)
-	(wire
-		(pts
 			(xy 144.78 69.85) (xy 143.51 69.85)
 		)
@@
 	(wire
 		(pts
-			(xy 158.75 110.49) (xy 140.97 110.49)
+			(xy 158.75 110.49) (xy 154.94 110.49)
 		)
 		(stroke
@@
 		(body_style 1)
 		(exclude_from_sim no)
-		(in_bom yes)
+		(in_bom no)
 		(on_board yes)
 		(in_pos_files yes)
