File: KiCAD/SensorBoard/SensorBoard.kicad_pcb (KiCad board)
At the start: 4 copper layers, 44 x 65 mm, 32 parts, among them J1 Conn_01x06_Pin, U1 AS7341DLG, U2 LSM9DS1, U3 VL53L0CXV0DH1, U4 AP7384-33V, U5 NCP1117-2.0_SOT223, U6 SC18IS604PW

Commit message: added a still, wip version of the sensor board
Parts:
- added D4: SK6805, LED_SMD:LED_SK6805_PLCC4_2.4x2.7mm_P1.3mm, B.Cu at (45.2, 61.9)
- added D5: SK6805, LED_SMD:LED_SK6805_PLCC4_2.4x2.7mm_P1.3mm, B.Cu at (23.0, 58.6)
- added D6: SK6805, LED_SMD:LED_SK6805_PLCC4_2.4x2.7mm_P1.3mm, B.Cu at (34.2, 60.1)
- added D7: LED, LED_SMD:LED_0805_2012Metric, B.Cu at (19.7, 70.2)
- added D8: LED, LED_SMD:LED_0805_2012Metric, B.Cu at (19.7, 72.2)
- added D9: LED, LED_SMD:LED_0805_2012Metric, B.Cu at (19.7, 74.2)
- added R7: 330, Resistor_SMD:R_0805_2012Metric, B.Cu at (14.6, 67.2)
- added R8: 330, Resistor_SMD:R_0805_2012Metric, B.Cu at (16.0, 70.1)
- added R9: 330, Resistor_SMD:R_0805_2012Metric, B.Cu at (13.8, 70.1)
- added U7: BMP280, Package_LGA:Bosch_LGA-8_2x2.5mm_P0.65mm_ClockwisePinNumbering, B.Cu at (20.8, 46.8)
- added U8: LM75B, Package_SO:SOIC-8_3.9x4.9mm_P1.27mm, B.Cu at (21.5, 33.6)
- moved G*** 18.0 mm to (33.0, 48.8)
Connections:
- D3 pad 1: unconnected-(D3-DOUT-Pad1) -> Net-(D3-DOUT)
Routing:
- net Net-(BZ1-+): track 216.0 -> 329.3 mm, vias 27 -> 37
- net Net-(D1-VDD): track 169.5 -> 234.8 mm, vias 18 -> 22
- net Net-(D7-A): track 67.3 -> 101.1 mm
- net Net-(D8-A): track 69.9 -> 103.6 mm, vias 3 -> 6
- net Net-(D1-DOUT): track 141.3 -> 174.6 mm, vias 13 -> 18
- net Net-(D4-DOUT): track 0.00 -> 30.8 mm, vias 0 -> 2
- net Net-(J1-Pin_3): track 109.0 -> 133.9 mm, vias 8 -> 11
- net Net-(D3-DOUT): track 0.00 -> 16.0 mm, vias 0 -> 1
- net Net-(D7-K): track 0.00 -> 11.9 mm, vias 0 -> 2
- net Net-(D8-K): track 0.00 -> 11.4 mm, vias 0 -> 2
- net Net-(D9-K): track 0.00 -> 11.1 mm, vias 0 -> 2
- net Net-(D5-DOUT): track 0.00 -> 10.4 mm, vias 0 -> 2
Other:
- board text added: "2V"
- board text added: "3V"
- board text added: "5V"

Commit message: updates to BOM and updates to othere boards (context of kicad pcbs)
Parts:
- added D10: LED, LED_SMD:LED_0805_2012Metric, F.Cu at (17.0, 20.8)
- added R10: 330, Resistor_SMD:R_0805_2012Metric, B.Cu at (17.0, 23.8)
- added U9: AS7341DLG, Package_LGA:AMS_OLGA-8_2x3.1mm_P0.8mm, F.Cu at (34.1, 53.8)
Routing:
- net Net-(D8-A): track 103.6 -> 140.4 mm, vias 6 -> 10
- net Net-(BZ1-+): track 329.3 -> 340.9 mm
- net Net-(BZ1--): track 64.5 -> 75.8 mm, vias 1 -> 3
- net Net-(D1-DOUT): track 174.6 -> 180.6 mm, vias 18 -> 20
- net Net-(D10-K): track 0.00 -> 3.02 mm, vias 0 -> 1
- net Net-(D1-VDD): track 234.8 -> 237.8 mm, vias 22 -> 25
- net Net-(J1-Pin_3): vias 11 -> 12
Other:
- board text added: "BUZZER"
- board text added: "UWB"
