File: KiCAD/SensorBoard/SensorBoard.kicad_sch (KiCad schematic)
At the start: 27 parts, among them J1 Conn_01x06_Pin, U1 AS7341DLG, U2 LSM9DS1, U3 VL53L0CXV0DH1, U4 AP7384-33V, U5 NCP1117-2.0_SOT223, U6 SC18IS604PW

Commit message: added a still, wip version of the sensor board
Parts:
- added D4, D5, D6: SK6805, LED_SMD:LED_SK6805_PLCC4_2.4x2.7mm_P1.3mm, symbol LED:SK6805
- added D7, D8, D9: LED, LED_SMD:LED_0805_2012Metric, symbol Device:LED
- added R7, R8, R9: 330, R_0805_2012Metric, symbol Device:R
- added U7: BMP280, Package_LGA:Bosch_LGA-8_2x2.5mm_P0.65mm_ClockwisePinNumbering, symbol Sensor_Pressure:BMP280
- added U8: LM75B, Package_SO:SOIC-8_3.9x4.9mm_P1.27mm, symbol Sensor_Temperature:LM75B
Connections:
- net at C1.1, C3.2, C4.2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: now also D4.4 (VDD), D5.4 (VDD), D6.4 (VDD), U7.2 (CSB), U7.6 (VDDIO), U7.8 (VDD), U8.8 (+Vs)
- net at BZ1.1 (+), C1.2, C2.2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: now also D4.2 (VSS), D5.2 (VSS), D6.2 (VSS), R7.2, R8.2, R9.2, U7.1 (GND), U7.5 (SDO), U7.7 (GND), U8.4 (GND), U8.5 (A2), U8.6 (A1), U8.7 (A0)
- net at C7.1, U1.1 (VDD), U5.2 (VO): now also D8.2 (A)
- net at J1.3 (Pin_3), R1.1, U1.2 (SCL)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: now also U7.4 (SCK), U8.2 (SCL)
- net at D1.1 (DOUT), D2.3 (DIN), J1.2 (Pin_2)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: now also U7.3 (SDI), U8.1 (SDA)
- net at C2.1, J1.1 (Pin_1), U3.5 (XSHUT)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: now also D7.2 (A), D9.2 (A)
- net at D3.1 (DOUT): now also D4.3 (DIN)
- new net: D7.1 (K), R7.1
- new net: D4.1 (DOUT), D5.3 (DIN)
- new net: D5.1 (DOUT), D6.3 (DIN)
- new net: D9.1 (K), R9.1
- new net: D8.1 (K), R8.1
- no-connect marks 27 -> 31

Commit message: updates to BOM and updates to othere boards (context of kicad pcbs)
Parts:
- added D10: LED, LED_SMD:LED_0805_2012Metric, symbol Device:LED
- added R10: 330, R_0805_2012Metric, symbol Device:R
- added U9: AS7341DLG, Package_LGA:AMS_OLGA-8_2x3.1mm_P0.8mm, symbol Sensor_Optical:AS7341DLG
Connections:
- net at BZ1.1 (+), C1.2, C2.2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: now also D10.2 (A), U9.3 (GND), U9.5 (PGND)
- net at C7.1, D8.2 (A), U1.1 (VDD)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: now also U9.1 (VDD)
- net at J1.3 (Pin_3), R1.1, U1.2 (SCL)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: now also U9.2 (SCL)
- net at D1.1 (DOUT), D2.3 (DIN), J1.2 (Pin_2)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: now also U9.8 (SDA)
- net at BZ1.2 (-), J1.4 (Pin_4): now also R10.2
- new net: D10.1 (K), R10.1
- no-connect marks 31 -> 35
