File: KiCAD/SensorSubmoduleFrontToF/SensorSubmoduleFrontToF.kicad_sch (KiCad schematic)
At the start: 6 parts, among them J1 Conn_01x04_Pin, U1 VL53L0CXV0DH1, U2 AP2112K-3.3

Commit message: updates to BOM and updates to othere boards (context of kicad pcbs)
Parts:
- R2, R3: footprint Resistor_SMD:R_01005_0402Metric -> Resistor_SMD:R_0603_1608Metric
Connections:
- net at R1.1, U1.11 (AVDD), U2.5 (VOUT): now also R2.1, R3.1
- net at J1.1 (Pin_1), U2.1 (VIN), U2.3 (EN): no longer R2.1, R3.1
Changed lines of the file:
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@@
 	(paper "A4")
+	(junction
+		(at 129.54 63.5)
+		(diameter 0)
+		(color 0 0 0 0)
+	)
 	(junction
 		(at 106.68 71.12)
@@
 	)
 	(junction
-		(at 129.54 60.96)
-		(diameter 0)
-		(color 0 0 0 0)
-	)
-	(junction
 		(at 132.08 76.2)
 		(diameter 0)
@@
 	(wire
 		(pts
-			(xy 125.73 71.12) (xy 125.73 66.04)
-		)
-		(stroke
-			(width 0)
-			(type default)
-		)
-	)
-	(wire
-		(pts
 			(xy 128.27 68.58) (xy 128.27 76.2)
 		)
@@
 	(wire
 		(pts
+			(xy 147.32 57.15) (xy 147.32 58.42)
+		)
+		(stroke
+			(width 0)
+			(type default)
+		)
+	)
+	(wire
+		(pts
+			(xy 127 71.12) (xy 127 91.44)
+		)
+		(stroke
+			(width 0)
+			(type default)
+		)
+	)
+	(wire
+		(pts
 			(xy 127 91.44) (xy 138.43 91.44)
 		)
@@
 	(wire
 		(pts
+			(xy 132.08 57.15) (xy 132.08 55.88)
+		)
+		(stroke
+			(width 0)
+			(type default)
+		)
+	)
+	(wire
+		(pts
 			(xy 114.3 60.96) (xy 114.3 63.5)
 		)
@@
 	(wire
 		(pts
-			(xy 125.73 66.04) (xy 127 66.04)
-		)
-		(stroke
-			(width 0)
-			(type default)
-		)
-	)
-	(wire
-		(pts
 			(xy 129.54 78.74) (xy 153.67 78.74)
 		)
@@
 	(wire
 		(pts
-			(xy 129.54 60.96) (xy 129.54 63.5)
+			(xy 132.08 63.5) (xy 129.54 63.5)
 		)
 		(stroke
@@
 	(wire
 		(pts
-			(xy 132.08 68.58) (xy 132.08 60.96)
-		)
-		(stroke
-			(width 0)
-			(type default)
-		)
-	)
-	(wire
-		(pts
 			(xy 138.43 68.58) (xy 138.43 91.44)
 		)
@@
 	(wire
 		(pts
+			(xy 129.54 63.5) (xy 129.54 57.15)
+		)
+		(stroke
+			(width 0)
+			(type default)
+		)
+	)
+	(wire
+		(pts
 			(xy 144.78 67.31) (xy 139.7 67.31)
 		)
@@
 	(wire
 		(pts
+			(xy 129.54 57.15) (xy 132.08 57.15)
+		)
+		(stroke
+			(width 0)
+			(type default)
+		)
+	)
+	(wire
+		(pts
 			(xy 163.83 91.44) (xy 166.37 91.44)
 		)
@@
 	(wire
 		(pts
-			(xy 114.3 60.96) (xy 129.54 60.96)
-		)
-		(stroke
-			(width 0)
-			(type default)
-		)
-	)
-	(wire
-		(pts
 			(xy 132.08 76.2) (xy 153.67 76.2)
 		)
@@
 	(wire
 		(pts
-			(xy 129.54 60.96) (xy 130.81 60.96)
+			(xy 114.3 60.96) (xy 130.81 60.96)
 		)
 		(stroke
@@
 	(wire
 		(pts
-			(xy 127 66.04) (xy 127 91.44)
-		)
-		(stroke
-			(width 0)
-			(type default)
-		)
-	)
-	(wire
-		(pts
-			(xy 106.68 71.12) (xy 125.73 71.12)
+			(xy 144.78 55.88) (xy 144.78 57.15)
+		)
+		(stroke
+			(width 0)
+			(type default)
+		)
+	)
+	(wire
+		(pts
+			(xy 106.68 71.12) (xy 127 71.12)
 		)
 		(stroke
@@
 	(wire
 		(pts
+			(xy 132.08 68.58) (xy 132.08 63.5)
+		)
+		(stroke
+			(width 0)
+			(type default)
+		)
+	)
+	(wire
+		(pts
 			(xy 163.83 58.42) (xy 163.83 60.96)
+		)
+		(stroke
+			(width 0)
+			(type default)
+		)
+	)
+	(wire
+		(pts
+			(xy 144.78 57.15) (xy 147.32 57.15)
+		)
+		(stroke
+			(width 0)
+			(type default)
+		)
+	)
+	(wire
+		(pts
+			(xy 132.08 55.88) (xy 144.78 55.88)
 		)
 		(stroke
@@
 			)
 		)
-		(property "Footprint" "Resistor_SMD:R_01005_0402Metric"
+		(property "Footprint" "Resistor_SMD:R_0603_1608Metric"
 			(at 127.762 67.31 90)
 			(hide yes)
@@
 		(exclude_from_sim no)
 		(in_bom no)
-		(on_board no)
+		(on_board yes)
 		(in_pos_files no)
 		(dnp no)
@@
 			)
 		)
-		(property "Footprint" "Resistor_SMD:R_01005_0402Metric"
+		(property "Footprint" "Resistor_SMD:R_0603_1608Metric"
 			(at 130.302 72.39 90)
 			(hide yes)
